File: hardware/megabank.kicad_pcb (KiCad board)
At the start: 4 copper layers, 130 x 56 mm, 89 parts, among them J1 USB-C, P1 TS2068_Edge, Q1 AO3401A, Q2 AO3400A, SW3 RUN, SW4 BOOTSEL, SW5 WP, U1 74LVC245APW, U10 CY62167EV30LL-45ZXIT, U11 CY62167EV30LL-45ZXIT, U12 SN74LVC1G32DBVR, U2 74LVC245APW, U20 RP2350B, U21 GD25Q128ESIGR, U3 74LVC245APW, U30 TLV1117LV33, U31 TPS3839G33, U32 LM66200, U4 74LVC245APW, U5 74LVC1G06, Y1 12MHz

Commit message: Board: battery holder and switch checked against drawings; re-routed
Battery holder: Keystone 3034's footprint was wrong for the Q&J
CR2032-BS-6-1 (C70377), which has a + tab at one end and a - tab at the
other. New project footprint from Q&J's drawing QJ.BS-6: two 4.2 x 3.0 mm
pads, 26 mm apart inside, 32 mm outside. BT1 turned 90 degrees to fit.

Slide switch: KiCad's MSK12C02 footprint matches the drawing. SW5 moved
right 2.1 mm so the actuator tip sits at the board edge.

Re-routing then left nets from the RP2350B's top pad row open, so
preroute.py now fans pins 42-48 (PA16-PA20, WINH, nWP) into lanes to the
right. For room, C27 moved up and BAT_ADC moved from GPIO40 to GPIO43
(ADC3). Routed by flow.py on its second attempt, DRC clean at every
severity: 1765 track segments, 320 vias.

Co-Authored-By: Claude Opus 5.5 <noreply@anthropic.com>
Parts:
- BT1: footprint BatteryHolder_Keystone_3034_1x20mm -> BatteryHolder_QJ_CR2032-BS-6-1
- moved C27 2.20 mm to (67.4, 15.2), turned to 0 degrees
- moved SW5 2.10 mm to (127.1, 41.0)
- moved BT1 0.81 mm to (20.1, 36.7), turned to 90 degrees
Connections:
- U20 pad 49: BAT_ADC -> unconnected-(U20-GPIO40/ADC0-Pad49)
- U20 pad 54: unconnected-(U20-GPIO43/ADC3-Pad54) -> BAT_ADC
Routing:
- net SD5: track 118.6 -> 144.4 mm
- net BA10: track 65.5 -> 86.3 mm
- net /RP2350B Controller/SWCLK: track 57.8 -> 37.8 mm, vias 4 -> 2
- net PA18: track 66.3 -> 85.8 mm, vias 4 -> 5
- net SD7: track 108.5 -> 127.5 mm, vias 3 -> 4
- net BA0: track 94.2 -> 113.1 mm
- net nRD_L: track 98.6 -> 114.7 mm
- net BA1: track 101.5 -> 86.4 mm, vias 2 -> 3
- net BA2: track 99.3 -> 85.1 mm, vias 0 -> 2
- net BA3: track 96.2 -> 82.5 mm, vias 2 -> 3
- net /RP2350B Controller/RUN: track 31.8 -> 43.7 mm
- net PA15: track 52.2 -> 63.7 mm, vias 2 -> 5
- net BA13: track 29.4 -> 40.5 mm
- net nWP: track 90.9 -> 80.8 mm, vias 6 -> 2
- net BA7: track 74.6 -> 84.5 mm, vias 4 -> 2
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