File: hardware/power.kicad_sch (KiCad schematic)
At the start: 19 parts, among them Q1 AO3401A, Q2 AO3400A, U30 TLV1117LV33, U31 TPS3839G33, U32 LM66200

Commit message: Board: battery holder and switch checked against drawings; re-routed
Battery holder: Keystone 3034's footprint was wrong for the Q&J
CR2032-BS-6-1 (C70377), which has a + tab at one end and a - tab at the
other. New project footprint from Q&J's drawing QJ.BS-6: two 4.2 x 3.0 mm
pads, 26 mm apart inside, 32 mm outside. BT1 turned 90 degrees to fit.

Slide switch: KiCad's MSK12C02 footprint matches the drawing. SW5 moved
right 2.1 mm so the actuator tip sits at the board edge.

Re-routing then left nets from the RP2350B's top pad row open, so
preroute.py now fans pins 42-48 (PA16-PA20, WINH, nWP) into lanes to the
right. For room, C27 moved up and BAT_ADC moved from GPIO40 to GPIO43
(ADC3). Routed by flow.py on its second attempt, DRC clean at every
severity: 1765 track segments, 320 vias.

Co-Authored-By: Claude Opus 5.5 <noreply@anthropic.com>
Parts:
- BT1: footprint Battery:BatteryHolder_Keystone_3034_1x20mm -> megabank:BatteryHolder_QJ_CR2032-BS-6-1
Changed lines of the file:
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@@
     (property "Reference" "BT1" (at 62.69 160.6 0) (effects (font (size 1.27 1.27)) (justify left)))
     (property "Value" "CR2032" (at 62.69 163.1 0) (effects (font (size 1.27 1.27)) (justify left)))
-    (property "Footprint" "Battery:BatteryHolder_Keystone_3034_1x20mm" (at 59.69 170.18 0) (effects (font (size 1.27 1.27)) (justify left) (hide yes)))
+    (property "Footprint" "megabank:BatteryHolder_QJ_CR2032-BS-6-1" (at 59.69 170.18 0) (effects (font (size 1.27 1.27)) (justify left) (hide yes)))
     (property "Datasheet" "" (at 59.69 170.18 0) (effects (font (size 1.27 1.27)) (justify left) (hide yes)))
     (property "Description" "" (at 59.69 170.18 0) (effects (font (size 1.27 1.27)) (justify left) (hide yes)))
