File: hardware/interface.kicad_sch (KiCad schematic)
At the start: 14 parts, among them P1 TS2068_Edge, U1 74LVC245APW, U2 74LVC245APW, U3 74LVC245APW, U4 74LVC245APW, U5 74LVC1G06

Commit message: Board: /INT and /NMI for the controller (open question 16)
- U7 SN74LVC2G34 brings /INT (A14) and /NMI (A15) to GPIO43/44.
- U6, a second 74LVC1G06, pulls /NMI from GPIO45 (NMI_REQ), open-drain
  like /BE; R4 holds NMI_REQ low until the firmware runs.
- Placed over fingers A14/A15 between C3 and U2. Re-routed by flow.py
  (closed on attempt 2): DRC clean, nothing unconnected; ERC has the one
  expected warning. BOMs and renders regenerated.
- Spec: pin table (46 of 48, now counting the /BE read-back), parts,
  open question 16 marked added.

Co-Authored-By: Claude Opus 5.5 <noreply@anthropic.com>
Parts:
- added C6, C7: 100n, Capacitor_SMD:C_0603_1608Metric, symbol Device:C
- added R4: 10k, Resistor_SMD:R_0603_1608Metric, symbol Device:R
- added U6: 74LVC1G06, Package_TO_SOT_SMD:SOT-353_SC-70-5, symbol 74xGxx:74LVC1G06
- added U7: 74LVC2G34, Package_TO_SOT_SMD:SOT-363_SC-70-6, symbol 74xGxx:74LVC2G34
Connections:
- net +3V3: now also C6.1, C7.1, U6.5 (VCC), U7.5 (VCC)
- net GND: now also C6.2, C7.2, R4.2, U6.3 (GND), U7.2 (GND)
- net nINT: now reaches P1.A14 (~{INT})
- net nINT: now also U7.1
- net nNMI: now reaches P1.A15 (~{NMI})
- net nNMI: now also U6.4, U7.3
- new net NMI_REQ: R4.1, U6.2
- new net nINT_L: U7.6
- new net nNMI_L: U7.4
- no-connect marks 23 -> 21
Other:
- note added: "U6: open drain, like U5; R4 holds NMI_REQ low (released) until the firmware runs."
- note added: "U7: /INT and /NMI in, for the controller (spec, open question 16). /NMI's pull-up is the 2068's."
